File: hardware/backlight/backlight.sch (EAGLE design)
At the start: 39 parts, among them J1 1x8 header, U1 ATTINY45-20SU

Commit message: thicken traces again
Parts:
- added U$17: CMD_C0DE_LOGOCMD_CODE_LOGO_TOP_COPPER, logos:CMD_C0DE_LOGOCMD_CODE_LOGO_TOP_COPPER
Changed lines of the file:
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@@
 <part name="C19" library="passives" deviceset="C-US" device="C0805K" package3d_urn="urn:adsk.eagle:package:8089589/1" value="15pF"/>
 <part name="R1" library="passives" deviceset="RESISTOR" device="R0805-RES" package3d_urn="urn:adsk.eagle:package:8118506/2" value="4.7K"/>
+<part name="U$17" library="logos" deviceset="CMD_C0DE_LOGO" device="CMD_CODE_LOGO_TOP_COPPER"/>
 </parts>
 <sheets>
@@
 <attribute name="VALUE" x="18.542" y="82.55" size="1.778" layer="96" rot="R90"/>
 </instance>
+<instance part="U$17" gate="G$1" x="45.72" y="12.7" smashed="yes"/>
 </instances>
 <busses>
